File: KiCAD/K68-SC1602.kicad_pcb (KiCad board)
At the start: 2 copper layers, 100 x 100 mm, 21 parts, among them J1 SBC8080 BUS, J2 I/O ADDR JP, J3 LCD_1列端子, J4 外部I/O端子-1, J5 LCD-2列端子, J6 外部I/O端子-2, SW1 LCD LIGHT SW, U1 74HC138, U2 74HC04, U3 74HC08

Commit message: REV1 基板データ ガーバー出力
Parts:
- J1: value SBC8080 BUS -> SBC68 BUS
- moved C1 68.7 mm to (184.4, 59.2)
Connections:
- net /$80 renamed /$8000-8003
- net /$90 renamed /$8004-8008
- net /$A0 renamed /$8008-800B
- net /$B0 renamed /$800C-800F
- net /$C0 renamed /$8010-8013
- net /$D0 renamed /$8014-8017
- net /$E0 renamed /$8018-801B
- net /$F0 renamed /$801C-801F
- J1 pad 1: VCC -> /~{RD}
- J1 pad 10: /D1 -> /D7
- J1 pad 11: /D2 -> /A0
- J1 pad 12: /D3 -> unconnected-(J1-Pin_12-Pad12)
- J1 pad 13: /D4 -> /A2
- J1 pad 14: /D5 -> /A3
- J1 pad 15: /D6 -> /A4
- J1 pad 16: /D7 -> unconnected-(J1-Pin_16-Pad16)
- J1 pad 17: /~{IOR} -> unconnected-(J1-Pin_17-Pad17)
- J1 pad 19: /~{IOW} -> unconnected-(J1-Pin_19-Pad19)
- J1 pad 2: GND -> /~{WR}
- J1 pad 25: /A0 -> unconnected-(J1-Pin_25-Pad25)
- J1 pad 26: /A1 -> /A15
- J1 pad 28: unconnected-(J1-Pin_28-Pad28) -> /E
- J1 pad 29: /A4 -> unconnected-(J1-Pin_29-Pad29)
- J1 pad 3: VCC -> /D0
- J1 pad 30: /A5 -> unconnected-(J1-Pin_30-Pad30)
- J1 pad 31: /A6 -> unconnected-(J1-Pin_31-Pad31)
- J1 pad 32: /A7 -> unconnected-(J1-Pin_32-Pad32)
- J1 pad 39: unconnected-(J1-Pin_39-Pad39) -> VCC
- J1 pad 4: GND -> /D1
- J1 pad 40: unconnected-(J1-Pin_40-Pad40) -> GND
- J1 pad 5: unconnected-(J1-Pin_5-Pad5) -> /D2
- J1 pad 6: unconnected-(J1-Pin_6-Pad6) -> /D3
- J1 pad 7: unconnected-(J1-Pin_7-Pad7) -> /D4
- J1 pad 8: unconnected-(J1-Pin_8-Pad8) -> /D5
- J1 pad 9: /D0 -> /D6
- RN1 pad 6: /A7 -> /A15
- RN1 pad 8: /A5 -> /A3
- RN1 pad 9: /A6 -> /A2
- U1 pad 1: /A6 -> /A2
- U1 pad 2: /A5 -> /A3
- U1 pad 4: GND -> /E
- U1 pad 6: /A7 -> /A15
- U3 pad 1: /~{IOR} -> /~{RD}
- U3 pad 2: /~{IOW} -> /~{WR}
Routing:
- net /A1: track 145.6 -> 86.7 mm
- net /A7: track 32.4 -> 0.00 mm
- net /A3: track 0.00 -> 29.1 mm
- net /~{IOW}: track 28.5 -> 0.00 mm
- net /A15: track 0.00 -> 27.9 mm
- net /A2: track 0.00 -> 26.4 mm
- net /~{IOR}: track 23.4 -> 0.00 mm
- net GND: track 304.7 -> 282.0 mm, vias 0 -> 1
- net /A5: track 21.2 -> 0.00 mm
- net /LCDSEL: track 138.9 -> 118.2 mm, vias 0 -> 1
- net /E: track 0.00 -> 20.2 mm
- net /~{WR}: track 0.00 -> 19.1 mm
- net /D0: track 134.3 -> 117.5 mm, vias 0 -> 1
- net /A6: track 15.2 -> 0.00 mm
- net /D2: track 140.5 -> 126.7 mm
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Other:
- board text added: "$00"
- board text added: "$04"
- board text added: "$08"
- board text added: "$0C"
- board text added: "$10"
- board text added: "$14"
- board text added: "$18"
- board text added: "$1C"
- board text added: "K68マイコン 液晶基板 REV1"
- board text added: "SBC68 バスコネクター"
- board text removed: "$80"
- board text removed: "$90"
- board text removed: "$A0"
- board text removed: "$B0"
- board text removed: "$C0"
- board text removed: "$D0"
- board text removed: "$E0"
- board text removed: "$F0"
- board text removed: "KZ80マイコン 液晶基板 REV1"
- board text removed: "SBC8080 バスコネクター"
