File: KiCAD/K68-SC1602.kicad_sch (KiCad schematic)
At the start: 21 parts, among them J1 SBC8080 BUS, J2 I/O ADDR JP, J3 LCD_1列端子, J4 外部I/O端子-1, J5 LCD-2列端子, J6 外部I/O端子-2, SW1 LCD LIGHT SW, U1 74HC138, U2 74HC04, U3 74HC08

Commit message: REV1 基板データ ガーバー出力
Parts:
- J1: value SBC8080 BUS -> SBC68 BUS
Connections:
- net A0: now also J1.11 (Pin_11); no longer J1.25 (Pin_25)
- net A1: no longer J1.26 (Pin_26)
- net A4: now also J1.15 (Pin_15); no longer J1.29 (Pin_29)
- net D0: now also J1.3 (Pin_3); no longer J1.9 (Pin_9)
- net D1: now also J1.4 (Pin_4); no longer J1.10 (Pin_10)
- net D2: now also J1.5 (Pin_5); no longer J1.11 (Pin_11)
- net D3: now also J1.6 (Pin_6); no longer J1.12 (Pin_12)
- net D4: now also J1.7 (Pin_7); no longer J1.13 (Pin_13)
- net D5: now also J1.8 (Pin_8); no longer J1.14 (Pin_14)
- net D6: now also J1.9 (Pin_9); no longer J1.15 (Pin_15)
- net D7: now also J1.10 (Pin_10); no longer J1.16 (Pin_16)
- net GND: now also J1.40 (Pin_40); no longer J1.2 (Pin_2), J1.4 (Pin_4), U1.4 (E1)
- net VCC: now also J1.39 (Pin_39); no longer J1.1 (Pin_1), J1.3 (Pin_3)
- net E: now reaches J1.28 (Pin_28)
- net E: now also U1.4 (E1)
- net $80 renamed $8000-8003
- net $90 renamed $8004-8008
- net $A0 renamed $8008-800B
- net $B0 renamed $800C-800F
- net $C0 renamed $8010-8013
- net $D0 renamed $8014-8017
- net $E0 renamed $8018-801B
- net $F0 renamed $801C-801F
- net A5 renamed A3
- net A3: now also J1.14 (Pin_14); no longer J1.30 (Pin_30)
- net A6 renamed A2
- net A2: now also J1.13 (Pin_13); no longer J1.31 (Pin_31)
- net A7 renamed A15
- net A15: now also J1.26 (Pin_26); no longer J1.32 (Pin_32)
- net ~{IOR}: no longer names the net of J1.17 (Pin_17)
- net ~{IOR}: no longer U3.1
- net ~{IOW}: no longer names the net of J1.19 (Pin_19)
- net ~{IOW}: no longer U3.2
- new net ~{RD}: J1.1 (Pin_1), U3.1
- new net ~{WR}: J1.2 (Pin_2), U3.2
- no-connect marks 47 -> 49
Other:
- title: KZ80 LCD SC1602 BOARD -> K68 LCD SC1602 BOARD
- moved on the sheet: C1, J2, U2A, U2B, U2C, U2D
